File: Eagle Board/Arduino Maple Uno.sch (EAGLE design)
At the start: 66 parts, among them T1 BC847, T2 BC847, U1 3.3V, U2 MCP9808MSOP, X1 8Mhz

Commit message: changes in design
Parts:
- removed U$4: 3015-INDUCTOR, LCSC:3015-INDUCTOR
- added C13: 100nF, resistor:C-EUC0603
- added U$6: 6045-3.6A-INDUCTOR, LCSC:6045-3.6A-INDUCTOR
- R11: value 56k -> 100k
- R12: value 10k -> 13.7k
- T1, T2: value BC847 -> S8050
- U$2: value ME3116 -> SY8113; device LCSC:ME3116 -> LCSC:SY8113
Connections:
- net 3.3V: now also C13.1; no longer LED2.A
- net 33: now also LED2.A; no longer R23.2
- net GND: now also C13.2, R23.2
- net N$24: now also U$6.2; no longer U$4.2
- net N$5: now also U$6.1; no longer U$4.1
Other:
- note added: "1.0"
- moved on the sheet: LED2, R23

Commit message: added MPU6050 IMU
Parts:
- added C19: 10nF, resistor:C-EUC0603
- added C20: 2.2nF, resistor:C-EUC0603
- added C21: 100nF, resistor:C-EUC0603
- added R25, R26: 10k, resistor:R-US_R0603
- added U$4: MPU-6050-1, LCSC:MPU-6050-1
Connections:
- new net N$33: C21.1, U$4.REGOUT
- new net N$35: C20.1, U$4.CPOUT
- net 20: now also U$4.INT
- net 3.3V: now also C19.1, R25.2, R26.2, U$4.VDD, U$4.VLOGIC; no longer LED1.A
- net GND: now also C19.2, C20.2, C21.2, R22.2, U$4.AD0, U$4.CLKIN, U$4.FSYNC, U$4.GND
- net N$20: now also C12.1, C17.1, D3.C, R10.2, U$2.VIN; no longer D3.A, U$3.TIP
- net PIO1: now also LED1.A; no longer R22.2
- net SCL: now also R25.1, U$4.SCL
- net SDA: now also R26.1, U$4.SDA
- net VIN: now also D3.A, U$3.TIP; no longer C12.1, C17.1, D3.C, R10.2, U$2.VIN
Other:
- note added: "SENSORS"
- note removed: "TEMP SENSOR"
- moved on the sheet: D3, R13, R14, R15, R16, R17, U$3, U2
